Commit message: robot redisign

File: Project2/catkin_ws/src/my_robot/urdf/macros.xacro (robot description, xacro)
@@ -7,3 +7,15 @@
     />
   </macro>
+  <macro name="cylinder_inertia" params="m r h">
+    <inertia  ixx="${m*(3*r*r+h*h)/12}" ixy = "0" ixz = "0"
+      iyy="${m*(3*r*r+h*h)/12}" iyz = "0"
+      izz="${m*r*r/2}"
+    />
+  </macro>
+  <macro name="sphere_inertia" params="m r">
+    <inertia  ixx="${2*m*r*r/5}" ixy = "0" ixz = "0"
+      iyy="${2*m*r*r/5}" iyz = "0"
+      izz="${2*m*r*r/5}"
+    />
+  </macro>
 </robot>

File: Project2/catkin_ws/src/my_robot/urdf/my_robot.xacro (robot description, xacro)
@@ -2,5 +2,18 @@
 <robot name="my_robot"
   xmlns:xacro="http://www.ros.org/wiki/xacro">
-  <!-- <xacro:include filename="$(find my_robot)/urdf/macros.xacro"/> -->
+  <xacro:property name="PI" value="3.1415926535897931"/>
+  <xacro:property name="chassisHeight" value="0.1"/>
+  <xacro:property name="chassisRadius" value="0.2"/>
+  <xacro:property name="chassisLength" value="${chassisRadius * 2}"/>
+  <xacro:property name="chassisMass" value="15"/>
+  <xacro:property name="casterRadius" value="0.0499"/>
+  <xacro:property name="casterMass" value="5"/>
+  <xacro:property name="wheelWidth" value="0.05"/>
+  <xacro:property name="wheelRadius" value="0.1"/>
+  <xacro:property name="wheelPos" value="${chassisRadius + wheelWidth}"/>
+  <xacro:property name="wheelMass" value="5"/>
+  <xacro:property name="cameraSize" value="0.05"/>
+  <xacro:property name="cameraMass" value="0.1"/>
+  <xacro:include filename="$(find my_robot)/urdf/macros.xacro"/>
   <xacro:include filename="$(find my_robot)/urdf/materials.gazebo"/>
   <xacro:include filename="$(find my_robot)/urdf/my_robot.gazebo" />
@@ -12,14 +25,14 @@
   </joint>
   <link name='chassis'>
-    <pose>0 0 0.1 0 0 0</pose>
+    <pose>0 0 0 0 0 0</pose>
     <inertial>
-      <mass value="15.0"/>
+      <mass value="${chassisMass}"/>
       <origin xyz="0.0 0 0" rpy=" 0 0 0"/>
-      <inertia ixx="0.1" ixy="0" ixz="0" iyy="0.1" iyz="0" izz="0.1" />
+      <cylinder_inertia m="${chassisMass}" r="${chassisRadius}" h="${chassisHeight}" />
     </inertial>
     <collision name='collision'>
       <origin xyz="0 0 0" rpy=" 0 0 0"/>
       <geometry>
-        <box size=".4 .2 .1"/>
+        <cylinder length="${chassisHeight}" radius="${chassisRadius}"/>
       </geometry>
     </collision>
@@ -27,38 +40,41 @@
       <origin xyz="0 0 0" rpy=" 0 0 0"/>
       <geometry>
-        <box size=".4 .2 .1"/>
+        <cylinder length="${chassisHeight}" radius="${chassisRadius}"/>
       </geometry>
     </visual>
+    <!-- caster wheels -->
+    <!-- back -->
     <collision name='back_caster_collision'>
-      <origin xyz="-0.15 0 -0.05" rpy=" 0 0 0"/>
+      <origin xyz="${casterRadius-chassisRadius} 0 ${chassisHeight - wheelRadius - casterRadius}" rpy=" 0 0 0"/>
       <geometry>
-        <sphere radius="0.0499"/>
+        <sphere radius="${casterRadius}"/>
       </geometry>
     </collision>
     <visual name='back_caster_visual'>
-      <origin xyz="-0.15 0 -0.05" rpy=" 0 0 0"/>
+      <origin xyz="${casterRadius-chassisRadius} 0 ${chassisHeight - wheelRadius - casterRadius}" rpy=" 0 0 0"/>
       <geometry>
-        <sphere radius="0.05"/>
+        <sphere radius="${casterRadius}"/>
       </geometry>
     </visual>
+    <!-- front -->
     <collision name='front_caster_collision'>
-      <origin xyz="0.15 0 -0.05" rpy=" 0 0 0"/>
+      <origin xyz="${chassisRadius - casterRadius} 0 ${chassisHeight - wheelRadius - casterRadius}" rpy=" 0 0 0"/>
       <geometry>
-        <sphere radius="0.0499"/>
+        <sphere radius="${casterRadius}"/>
       </geometry>
     </collision>
     <visual name='front_caster_visual'>
-      <origin xyz="0.15 0 -0.05" rpy=" 0 0 0"/>
+      <origin xyz="${chassisRadius - casterRadius} 0 ${chassisHeight - wheelRadius - casterRadius}" rpy=" 0 0 0"/>
       <geometry>
-        <sphere radius="0.05"/>
+        <sphere radius="${casterRadius}"/>
       </geometry>
     </visual>
   </link>
   <link name="left_wheel">
-   <pose>0 0.15 0 0 0 0</pose>
+   <pose>0 ${wheelPos} 0 0 0 0</pose>
     <visual>
       <origin xyz="0 0 0" rpy= "0 1.5707 1.5707"/>
       <geometry>
-        <cylinder radius="0.1" length="0.05"></cylinder>
+        <cylinder radius="${wheelRadius}" length="${wheelWidth}" />
       </geometry>
     </visual>
@@ -66,19 +82,19 @@
       <origin xyz="0 0 0" rpy= "0 1.5707 1.5707"/>
       <geometry>
-        <cylinder radius="0.1" length="0.05" />
+        <cylinder radius="${wheelRadius}" length="${wheelWidth}" />
       </geometry>
     </collision>
     <inertial>
-      <mass value="5.0"/>
+      <mass value="${wheelMass}"/>
       <origin xyz="0.0 0 0" rpy=" 0 1.5707 1.5707"/>
-      <inertia ixx="0.1" ixy="0" ixz="0" iyy="0.1" iyz="0" izz="0.1" />
+      <cylinder_inertia m="${wheelMass}" r="${wheelRadius}" h="${wheelWidth}" />
     </inertial>
   </link>
   <link name="right_wheel">
-    <pose>0 -0.15 0 0 0 0</pose>
+    <pose>0 ${-wheelPos} 0 0 0 0</pose>
     <visual>
       <origin xyz="0 0 0" rpy= "0 1.5707 1.5707"/>
       <geometry>
-        <cylinder radius="0.1" length="0.05"></cylinder>
+        <cylinder radius="${wheelRadius}" length="${wheelWidth}" />
       </geometry>
     </visual>
@@ -86,5 +102,5 @@
       <origin xyz="0 0 0" rpy= "0 1.5707 1.5707"/>
       <geometry>
-        <cylinder radius="0.1" length="0.05" />
+        <cylinder radius="${wheelRadius}" length="${wheelWidth}" />
       </geometry>
     </collision>
@@ -92,9 +108,9 @@
       <mass value="5.0"/>
        <origin xyz="0 0 0" rpy= "0 1.5707 1.5707"/>
-      <inertia ixx="0.1" ixy="0" ixz="0" iyy="0.1" iyz="0" izz="0.1" />
+       <cylinder_inertia m="${wheelMass}" r="${wheelRadius}" h="${wheelWidth}" />
     </inertial>
   </link>
  <joint type="continuous" name="left_wheel_hinge">
-    <origin xyz="0 0.15 0" rpy="0 0 0"/>
+    <origin xyz="0 ${wheelPos} 0" rpy="0 0 0"/>
     <child link="left_wheel"/>
     <parent link="chassis"/>
@@ -104,5 +120,5 @@
   </joint>
  <joint type="continuous" name="right_wheel_hinge">
-    <origin xyz="0 -0.15 0" rpy="0 0 0"/>
+    <origin xyz="0 ${-wheelPos} 0" rpy="0 0 0"/>
     <child link="right_wheel"/>
     <parent link="chassis"/>
@@ -116,5 +132,5 @@
       <origin xyz="0 0 0" rpy="0 0 0"/>
       <geometry>
-        <box size=".05 .05 .05"/>
+        <box size="${cameraSize} ${cameraSize} ${cameraSize}"/>
       </geometry>
     </collision>
@@ -122,17 +138,16 @@
       <origin xyz="0 0 0" rpy="0 0 0"/>
       <geometry>
-        <box size=".05 .05 .05"/>
+        <box size="${cameraSize} ${cameraSize} ${cameraSize}"/>
       </geometry>
     </visual>
-    <box_inertia x="0.05" y="0.05" z="0.05" m="0.1" />
     <inertial>
-      <mass value="0.1"/>
+      <mass value="${cameraMass}"/>
       <origin xyz="0.0 0.0 0.0" rpy="0.0 0.0 0.0"/>
-      <inertia ixx="1e-6" ixy="0.0" ixz="0.0" iyy="1e-6" iyz="0.0" izz="1e-6"/>
+      <box_inertia x="${cameraSize}" y="${cameraSize}" z="${cameraSize}" m="${cameraMass}" />
     </inertial>
   </link>
   <joint name="camera_joint" type="fixed">
     <axis xyz="0.0 1.0 0.0"/>
-    <origin xyz="0.2 0.0 0.0" rpy="0.0 0.0 0.0"/>
+    <origin xyz="${chassisRadius} 0.0 0.0" rpy="0.0 0.0 0.0"/>
     <parent link="chassis"/>
     <child link="camera"/>
