Commit message: lecture 8

File: Project2/catkin_ws/src/my_robot/urdf/my_robot.xacro (robot description, xacro)
@@ -2,4 +2,7 @@
 <robot name="my_robot"
   xmlns:xacro="http://www.ros.org/wiki/xacro">
+  <!-- <xacro:include filename="$(find my_robot)/urdf/macros.xacro"/> -->
+  <xacro:include filename="$(find my_robot)/urdf/materials.gazebo"/>
+  <xacro:include filename="$(find my_robot)/urdf/my_robot.gazebo" />
   <link name="robot_footprint"></link>
   <joint name="robot_footprint_joint" type="fixed">
@@ -108,3 +111,55 @@
     <dynamics damping="1.0" friction="1.0"/>
   </joint>
+  <link name="camera">
+    <origin xyz="0.0 0.0 0.0" rpy="0.0 0.0 0.0"/>
+    <collision name='collision'>
+      <origin xyz="0 0 0" rpy="0 0 0"/>
+      <geometry>
+        <box size=".05 .05 .05"/>
+      </geometry>
+    </collision>
+    <visual name='camera_visual'>
+      <origin xyz="0 0 0" rpy="0 0 0"/>
+      <geometry>
+        <box size=".05 .05 .05"/>
+      </geometry>
+    </visual>
+    <box_inertia x="0.05" y="0.05" z="0.05" m="0.1" />
+    <inertial>
+      <mass value="0.1"/>
+      <origin xyz="0.0 0.0 0.0" rpy="0.0 0.0 0.0"/>
+      <inertia ixx="1e-6" ixy="0.0" ixz="0.0" iyy="1e-6" iyz="0.0" izz="1e-6"/>
+    </inertial>
+  </link>
+  <joint name="camera_joint" type="fixed">
+    <axis xyz="0.0 1.0 0.0"/>
+    <origin xyz="0.2 0.0 0.0" rpy="0.0 0.0 0.0"/>
+    <parent link="chassis"/>
+    <child link="camera"/>
+  </joint>
+  <link name="hokuyo">
+    <inertial>
+      <origin xyz="0.0 0.0 0.0" rpy="0.0 0.0 0.0"/>
+      <mass value="1e-5"/>
+      <inertia ixx="1e-6" ixy="0.0" ixz="0.0" iyy="1e-6" iyz="0.0" izz="1e-6"/>
+    </inertial>
+    <visual name="hokuyo_visual">
+      <origin xyz="0.0 0.0 0.0" rpy="0.0 0.0 0.0"/>
+      <geometry>
+        <mesh filename="package://my_robot/meshes/hokuyo.dae"/>
+      </geometry>
+    </visual>
+    <collision name="hokuyo_collision">
+      <origin xyz="0.0 0.0 0.0" rpy="0.0 0.0 0.0"/>
+      <geometry>
+        <box size="0.1 0.1 0.1"/>
+      </geometry>
+    </collision>
+  </link>
+  <joint name="hokuyo_joint" type="fixed">
+    <origin xyz="0.15 0.0 0.1" rpy="0.0 0.0 0.0"/>
+    <parent link="chassis"/>
+    <child link="hokuyo"/>
+    <axis xyz="0.0 1.0 0.0"/>
+  </joint>
 </robot>

Commit message: cleanup xacro

File: Project2/catkin_ws/src/my_robot/urdf/my_robot.xacro (robot description, xacro)
@@ -5,12 +5,11 @@
   <xacro:property name="chassisHeight" value="0.1"/>
   <xacro:property name="chassisRadius" value="0.2"/>
-  <xacro:property name="chassisLength" value="${chassisRadius * 2}"/>
   <xacro:property name="chassisMass" value="15"/>
-  <xacro:property name="casterRadius" value="0.0499"/>
-  <xacro:property name="casterMass" value="5"/>
   <xacro:property name="wheelWidth" value="0.05"/>
   <xacro:property name="wheelRadius" value="0.1"/>
   <xacro:property name="wheelPos" value="${chassisRadius + wheelWidth}"/>
   <xacro:property name="wheelMass" value="5"/>
+  <xacro:property name="casterRadius" value="${wheelRadius / 2.0 - 0.0001}"/>
+  <xacro:property name="casterMass" value="5"/>
   <xacro:property name="cameraSize" value="0.05"/>
   <xacro:property name="cameraMass" value="0.1"/>

Commit message: xacro cleanup

File: Project2/catkin_ws/src/my_robot/urdf/my_robot.xacro (robot description, xacro)
@@ -8,7 +8,7 @@
   <xacro:property name="wheelWidth" value="0.05"/>
   <xacro:property name="wheelRadius" value="0.1"/>
-  <xacro:property name="wheelPos" value="${chassisRadius + wheelWidth}"/>
+  <xacro:property name="wheelPos" value="${chassisRadius + wheelWidth/2}"/>
   <xacro:property name="wheelMass" value="5"/>
-  <xacro:property name="casterRadius" value="${wheelRadius / 2.0 - 0.0001}"/>
+  <xacro:property name="casterRadius" value="${wheelRadius / 2.0}"/>
   <xacro:property name="casterMass" value="5"/>
   <xacro:property name="cameraSize" value="0.05"/>
@@ -27,9 +27,7 @@
     <inertial>
       <mass value="${chassisMass}"/>
-      <origin xyz="0.0 0 0" rpy=" 0 0 0"/>
       <cylinder_inertia m="${chassisMass}" r="${chassisRadius}" h="${chassisHeight}" />
     </inertial>
     <collision name='collision'>
-      <origin xyz="0 0 0" rpy=" 0 0 0"/>
       <geometry>
         <cylinder length="${chassisHeight}" radius="${chassisRadius}"/>
@@ -37,5 +35,4 @@
     </collision>
     <visual name='chassis_visual'>
-      <origin xyz="0 0 0" rpy=" 0 0 0"/>
       <geometry>
         <cylinder length="${chassisHeight}" radius="${chassisRadius}"/>
@@ -45,26 +42,26 @@
     <!-- back -->
     <collision name='back_caster_collision'>
-      <origin xyz="${casterRadius-chassisRadius} 0 ${chassisHeight - wheelRadius - casterRadius}" rpy=" 0 0 0"/>
+      <origin xyz="${casterRadius-chassisRadius} 0 ${-casterRadius}" rpy=" 0 0 0"/>
       <geometry>
-        <sphere radius="${casterRadius}"/>
+        <sphere radius="${casterRadius - 0.0001}"/>
       </geometry>
     </collision>
     <visual name='back_caster_visual'>
-      <origin xyz="${casterRadius-chassisRadius} 0 ${chassisHeight - wheelRadius - casterRadius}" rpy=" 0 0 0"/>
+      <origin xyz="${casterRadius-chassisRadius} 0 ${-casterRadius}" rpy=" 0 0 0"/>
       <geometry>
-        <sphere radius="${casterRadius}"/>
+        <sphere radius="${casterRadius - 0.0001}"/>
       </geometry>
     </visual>
     <!-- front -->
     <collision name='front_caster_collision'>
-      <origin xyz="${chassisRadius - casterRadius} 0 ${chassisHeight - wheelRadius - casterRadius}" rpy=" 0 0 0"/>
+      <origin xyz="${chassisRadius - casterRadius} 0 ${-casterRadius}" rpy=" 0 0 0"/>
       <geometry>
-        <sphere radius="${casterRadius}"/>
+        <sphere radius="${casterRadius - 0.0001}"/>
       </geometry>
     </collision>
     <visual name='front_caster_visual'>
-      <origin xyz="${chassisRadius - casterRadius} 0 ${chassisHeight - wheelRadius - casterRadius}" rpy=" 0 0 0"/>
+      <origin xyz="${chassisRadius - casterRadius} 0 ${-casterRadius}" rpy=" 0 0 0"/>
       <geometry>
-        <sphere radius="${casterRadius}"/>
+        <sphere radius="${casterRadius - 0.0001}"/>
       </geometry>
     </visual>

Commit message: cleanup urdf

File: Project2/catkin_ws/src/my_robot/urdf/my_robot.xacro (robot description, xacro)
@@ -3,14 +3,14 @@
   xmlns:xacro="http://www.ros.org/wiki/xacro">
   <xacro:property name="PI" value="3.1415926535897931"/>
-  <xacro:property name="chassisHeight" value="0.1"/>
-  <xacro:property name="chassisRadius" value="0.2"/>
+  <xacro:property name="chassisHeight" value="0.2"/>
+  <xacro:property name="chassisRadius" value="0.4"/>
   <xacro:property name="chassisMass" value="15"/>
-  <xacro:property name="wheelWidth" value="0.05"/>
-  <xacro:property name="wheelRadius" value="0.1"/>
+  <xacro:property name="wheelWidth" value="0.08"/>
+  <xacro:property name="wheelRadius" value="0.2"/>
   <xacro:property name="wheelPos" value="${chassisRadius + wheelWidth/2}"/>
   <xacro:property name="wheelMass" value="5"/>
   <xacro:property name="casterRadius" value="${wheelRadius / 2.0}"/>
   <xacro:property name="casterMass" value="5"/>
-  <xacro:property name="cameraSize" value="0.05"/>
+  <xacro:property name="cameraSize" value="0.1"/>
   <xacro:property name="cameraMass" value="0.1"/>
   <xacro:include filename="$(find my_robot)/urdf/macros.xacro"/>
@@ -151,10 +151,8 @@
   <link name="hokuyo">
     <inertial>
-      <origin xyz="0.0 0.0 0.0" rpy="0.0 0.0 0.0"/>
       <mass value="1e-5"/>
       <inertia ixx="1e-6" ixy="0.0" ixz="0.0" iyy="1e-6" iyz="0.0" izz="1e-6"/>
     </inertial>
     <visual name="hokuyo_visual">
-      <origin xyz="0.0 0.0 0.0" rpy="0.0 0.0 0.0"/>
       <geometry>
         <mesh filename="package://my_robot/meshes/hokuyo.dae"/>
@@ -162,5 +160,4 @@
     </visual>
     <collision name="hokuyo_collision">
-      <origin xyz="0.0 0.0 0.0" rpy="0.0 0.0 0.0"/>
       <geometry>
         <box size="0.1 0.1 0.1"/>
@@ -169,5 +166,5 @@
   </link>
   <joint name="hokuyo_joint" type="fixed">
-    <origin xyz="0.15 0.0 0.1" rpy="0.0 0.0 0.0"/>
+    <origin xyz="${7 * chassisRadius / 8.0} 0.0 0.15" rpy="0.0 0.0 0.0"/>
     <parent link="chassis"/>
     <child link="hokuyo"/>

Commit message: adding head

File: Project2/catkin_ws/src/my_robot/urdf/my_robot.xacro (robot description, xacro)
@@ -2,4 +2,5 @@
 <robot name="my_robot"
   xmlns:xacro="http://www.ros.org/wiki/xacro">
+  <!-- Properties -->
   <xacro:property name="PI" value="3.1415926535897931"/>
   <xacro:property name="chassisHeight" value="0.2"/>
@@ -14,4 +15,7 @@
   <xacro:property name="cameraSize" value="0.1"/>
   <xacro:property name="cameraMass" value="0.1"/>
+  <xacro:property name="headRadius" value="${chassisHeight}" />
+  <xacro:property name="headMass" value="${chassisMass / 3.0}" />
+  <!-- Includes -->
   <xacro:include filename="$(find my_robot)/urdf/macros.xacro"/>
   <xacro:include filename="$(find my_robot)/urdf/materials.gazebo"/>
@@ -67,4 +71,5 @@
     </visual>
   </link>
+  <!-- Wheels -->
   <link name="left_wheel">
    <pose>0 ${wheelPos} 0 0 0 0</pose>
@@ -123,4 +128,5 @@
     <dynamics damping="1.0" friction="1.0"/>
   </joint>
+  <!-- Sensors -->
   <link name="camera">
     <origin xyz="0.0 0.0 0.0" rpy="0.0 0.0 0.0"/>
@@ -171,3 +177,26 @@
     <axis xyz="0.0 1.0 0.0"/>
   </joint>
+  <link name="robot_head">
+    <pose>0.0 0.0 ${chassisHeight/2} 0.0 0.0 0.0</pose>
+    <inertial>
+      <mass value="${headMass}"/>
+      <sphere_inertia m="${headMass}" r="${headRadius}"/>
+    </inertial>
+    <visual>
+      <geometry>
+        <sphere radius="${headRadius}"/>
+      </geometry>
+    </visual>
+    <collision>
+      <geometry>
+        <sphere radius="${headRadius}"/>
+      </geometry>
+    </collision>
+  </link>
+  <joint name="joint_chassis_head" type="fixed">
+    <origin xyz="0.0 0.0 ${chassisHeight/2}" rpy="0.0 0.0 0.0"/>
+    <parent link="chassis"/>
+    <child link="robot_head"/>
+    <axis xyz="0.0 1 0.0"/>
+  </joint>
 </robot>
