Commit message: configs

File: Project3/catkin_ws/src/my_robot/urdf/my_robot.xacro (robot description, xacro)
@@ -151,5 +151,5 @@
   <joint name="camera_joint" type="fixed">
     <axis xyz="0.0 1.0 0.0"/>
-    <origin xyz="${chassisRadius} 0.0 0.0" rpy="0.0 0.0 0.0"/>
+    <origin xyz="${chassisRadius} -0.1 0.0" rpy="0.0 0.0 0.0"/>
     <parent link="chassis"/>
     <child link="camera"/>
@@ -172,5 +172,5 @@
   </link>
   <joint name="hokuyo_joint" type="fixed">
-    <origin xyz="${7 * chassisRadius / 8.0} 0.0 0.15" rpy="0.0 0.0 0.0"/>
+    <origin xyz="${chassisRadius} 0.1 0.0" rpy="0.0 0.0 0.0"/>
     <parent link="chassis"/>
     <child link="hokuyo"/>

Commit message: config fixes, sensor repositioning

File: Project3/catkin_ws/src/my_robot/urdf/my_robot.xacro (robot description, xacro)
@@ -151,5 +151,5 @@
   <joint name="camera_joint" type="fixed">
     <axis xyz="0.0 1.0 0.0"/>
-    <origin xyz="${chassisRadius} -0.1 0.0" rpy="0.0 0.0 0.0"/>
+    <origin xyz="${chassisRadius} -0.05 0.0" rpy="0.0 0.0 0.0"/>
     <parent link="chassis"/>
     <child link="camera"/>
@@ -172,5 +172,5 @@
   </link>
   <joint name="hokuyo_joint" type="fixed">
-    <origin xyz="${chassisRadius} 0.1 0.0" rpy="0.0 0.0 0.0"/>
+    <origin xyz="${chassisRadius} 0.05 0.0" rpy="0.0 0.0 0.0"/>
     <parent link="chassis"/>
     <child link="hokuyo"/>
