Commit message: fixing macros/typos

File: Project5/catkin_ws/src/my_robot/urdf/macros.xacro (robot description, xacro)
@@ -1,21 +1,21 @@
 <?xml version='1.0'?>
-<robot name="macros">
-  <macro name="box_inertia" params="m x y z">
+<robot name="xacro:macros" xmlns:xacro="http://www.ros.org/wiki/xacro">
+  <xacro:macro name="box_inertia" params="m x y z">
     <inertia  ixx="${m*(y*y+z*z)/12}" ixy = "0" ixz = "0"
       iyy="${m*(x*x+z*z)/12}" iyz = "0"
       izz="${m*(x*x+z*z)/12}"
     />
-  </macro>
-  <macro name="cylinder_inertia" params="m r h">
+  </xacro:macro>
+  <xacro:macro name="cylinder_inertia" params="m r h">
     <inertia  ixx="${m*(3*r*r+h*h)/12}" ixy = "0" ixz = "0"
       iyy="${m*(3*r*r+h*h)/12}" iyz = "0"
       izz="${m*r*r/2}"
     />
-  </macro>
-  <macro name="sphere_inertia" params="m r">
+  </xacro:macro>
+  <xacro:macro name="sphere_inertia" params="m r">
     <inertia  ixx="${2*m*r*r/5}" ixy = "0" ixz = "0"
       iyy="${2*m*r*r/5}" iyz = "0"
       izz="${2*m*r*r/5}"
     />
-  </macro>
+  </xacro:macro>
 </robot>

File: Project5/catkin_ws/src/my_robot/urdf/my_robot.xacro (robot description, xacro)
@@ -31,5 +31,5 @@
     <inertial>
       <mass value="${chassisMass}"/>
-      <cylinder_inertia m="${chassisMass}" r="${chassisRadius}" h="${chassisHeight}" />
+      <xacro:cylinder_inertia m="${chassisMass}" r="${chassisRadius}" h="${chassisHeight}" />
     </inertial>
     <collision name='collision'>
@@ -89,5 +89,5 @@
       <mass value="${wheelMass}"/>
       <origin xyz="0.0 0 0" rpy=" 0 1.5707 1.5707"/>
-      <cylinder_inertia m="${wheelMass}" r="${wheelRadius}" h="${wheelWidth}" />
+      <xacro:cylinder_inertia  m="${wheelMass}" r="${wheelRadius}" h="${wheelWidth}" />
     </inertial>
   </link>
@@ -109,5 +109,5 @@
       <mass value="5.0"/>
        <origin xyz="0 0 0" rpy= "0 1.5707 1.5707"/>
-       <cylinder_inertia m="${wheelMass}" r="${wheelRadius}" h="${wheelWidth}" />
+       <xacro:cylinder_inertia m="${wheelMass}" r="${wheelRadius}" h="${wheelWidth}" />
     </inertial>
   </link>
@@ -146,5 +146,5 @@
       <mass value="${cameraMass}"/>
       <origin xyz="0.0 0.0 0.0" rpy="0.0 0.0 0.0"/>
-      <box_inertia x="${cameraSize}" y="${cameraSize}" z="${cameraSize}" m="${cameraMass}" />
+      <xacro:box_inertia x="${cameraSize}" y="${cameraSize}" z="${cameraSize}" m="${cameraMass}" />
     </inertial>
   </link>
@@ -190,5 +190,5 @@
     <inertial>
       <mass value="${headMass}"/>
-      <sphere_inertia m="${headMass}" r="${headRadius}"/>
+      <xacro:sphere_inertia m="${headMass}" r="${headRadius}"/>
     </inertial>
     <visual>
