Commit message: populating rtab packages

File: Project5/catkin_ws/src/my_robot/urdf/my_robot.xacro (robot description, xacro)
@@ -128,5 +128,5 @@
     <dynamics damping="1.0" friction="1.0"/>
   </joint>
-  <!-- Sensors -->
+  <!-- Camera Sensor -->
   <link name="camera">
     <origin xyz="0.0 0.0 0.0" rpy="0.0 0.0 0.0"/>
@@ -155,4 +155,13 @@
     <child link="camera"/>
   </joint>
+  <!-- Optical Camera Sensor-->
+  <joint name="camera_optical_joint" type="fixed">
+    <origin xyz="0 0 0" rpy="-1.5707 0 -1.5707"/>
+    <parent link="camera_link"/>
+    <child link="camera_link_optical"/>
+  </joint>
+  <link name="camera_link_optical">
+  </link>
+  <!-- Laser Sensor-->
   <link name="hokuyo">
     <inertial>

Commit message: moving sensors around

File: Project5/catkin_ws/src/my_robot/urdf/my_robot.xacro (robot description, xacro)
@@ -151,5 +151,5 @@
   <joint name="camera_joint" type="fixed">
     <axis xyz="0.0 1.0 0.0"/>
-    <origin xyz="${chassisRadius} -0.05 0.0" rpy="0.0 0.0 0.0"/>
+    <origin xyz="${chassisRadius} 0.0 0.0" rpy="0.0 0.0 0.0"/>
     <parent link="chassis"/>
     <child link="camera"/>
@@ -181,5 +181,5 @@
   </link>
   <joint name="hokuyo_joint" type="fixed">
-    <origin xyz="${chassisRadius} 0.05 0.0" rpy="0.0 0.0 0.0"/>
+    <origin xyz="${chassisRadius - 0.05} 0 0.1" rpy="0.0 0.0 0.0"/>
     <parent link="chassis"/>
     <child link="hokuyo"/>

Commit message: working project

File: Project5/catkin_ws/src/my_robot/urdf/my_robot.xacro (robot description, xacro)
@@ -158,5 +158,5 @@
   <joint name="camera_optical_joint" type="fixed">
     <origin xyz="0 0 0" rpy="-1.5707 0 -1.5707"/>
-    <parent link="camera_link"/>
+    <parent link="camera"/>
     <child link="camera_link_optical"/>
   </joint>
